File: projects/msx_keyboard/msx_keyboard.kicad_pcb (KiCad board)
At the start: 2 copper layers, 505.5 x 190.5 mm, 111 parts, among them J1 Conn_01x04_Pin, J2 Conn_01x08_Pin, U1 4515

Commit message: Updated
Parts:
- added D12: CAPS_LED, LED_THT:LED_D5.0mm, F.Cu at (441.1, 88.4)
- added D13: KANA_LED, LED_THT:LED_D5.0mm, F.Cu at (453.8, 88.4)
- added G***: LOGO, 0-My_Parts:msx_logo, F.Cu at (82.6, 86.4)
- added G***: LOGO, 0-My_Parts:usa, F.Cu at (536.3, 246.0)
- added J3: Conn_01x01_Pin, Connector_PinSocket_2.54mm:PinSocket_1x01_P2.54mm_Vertical, F.Cu at (128.3, 79.6)
- added J4: Conn_01x01_Pin, Connector_PinSocket_2.54mm:PinSocket_1x01_P2.54mm_Vertical, F.Cu at (135.7, 79.6)
- added J5: Conn_01x02_Pin, Connector_PinHeader_2.54mm:PinHeader_1x02_P2.54mm_Vertical, F.Cu at (117.5, 79.6)
- added R10: R, Resistor_THT:R_Axial_DIN0207_L6.3mm_D2.5mm_P7.62mm_Horizontal, F.Cu at (527.6, 90.6)
- added R9: R, Resistor_THT:R_Axial_DIN0207_L6.3mm_D2.5mm_P7.62mm_Horizontal, F.Cu at (523.6, 90.6)
Routing:
- net Net-(D13-K): track 0.00 -> 325.3 mm, vias 0 -> 1
- net Net-(D12-K): track 0.00 -> 318.9 mm, vias 0 -> 1
- net VCC: track 322.6 -> 444.0 mm
- net GND: track 17.5 -> 114.7 mm, vias 0 -> 2
- net Net-(D12-A): track 0.00 -> 88.2 mm
- net Net-(D13-A): track 0.00 -> 71.1 mm
- net Net-(D6-A): track 332.8 -> 315.7 mm
- net /X4: track 843.9 -> 829.6 mm
- net /X7: track 801.0 -> 790.5 mm
- net /X2: track 768.4 -> 761.2 mm
- net Net-(D2-A): track 277.7 -> 271.1 mm
- net Net-(D3-A): track 457.1 -> 451.1 mm
- net /X6: track 750.9 -> 745.8 mm
- net /X0: track 886.4 -> 881.4 mm
- net Net-(D1-A): track 275.0 -> 270.3 mm
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
Commit message: Updated
Parts:
- added C1: C, Capacitor_THT:C_Disc_D3.0mm_W1.6mm_P2.50mm, F.Cu at (205.7, 87.4)
- added REF**: MountingHole_3.2mm_M3, MountingHole:MountingHole_3.2mm_M3, F.Cu at (221.0, 115.8)
- added REF**: MountingHole_3.2mm_M3, MountingHole:MountingHole_3.2mm_M3, F.Cu at (389.6, 244.7)
- added REF**: MountingHole_3.2mm_M3, MountingHole:MountingHole_3.2mm_M3, F.Cu at (547.3, 245.4)
- added REF**: MountingHole_3.2mm_M3, MountingHole:MountingHole_3.2mm_M3, F.Cu at (547.1, 86.7)
- added REF**: MountingHole_3.2mm_M3, MountingHole:MountingHole_3.2mm_M3, F.Cu at (63.7, 245.2)
- added REF**: MountingHole_3.2mm_M3, MountingHole:MountingHole_3.2mm_M3, F.Cu at (63.9, 86.7)
- added REF**: MountingHole_3.2mm_M3, MountingHole:MountingHole_3.2mm_M3, F.Cu at (388.7, 92.5)
- added REF**: MountingHole_3.2mm_M3, MountingHole:MountingHole_3.2mm_M3, F.Cu at (255.0, 245.1)
- SW_0, SW_1, SW_2, SW_3, SW_4, SW_5, SW_6, SW_7, SW_8, SW_9, SW_A1, SW_ASTA1, SW_AT1, SW_B1, SW_BS1, SW_C1, SW_CAPS1, SW_D1, SW_DOWN1, SW_E1, SW_ESC1, SW_F6, SW_G1, SW_GRP1, SW_GT1, SW_H1, SW_HAT1, SW_I1, SW_J1, SW_K1, SW_KANA1, SW_L1, SW_LBRAC1, SW_LEFT1, SW_LT1, SW_M1, SW_MINUS1, SW_N1, SW_O1, SW_P1, SW_PLUS1, SW_Q1, SW_R1, SW_RBRAC1, SW_RIGHT1, SW_S1, SW_SLASH1, SW_T0, SW_T1, SW_T10, SW_T2, SW_T3, SW_T4, SW_T5, SW_T6, SW_T7, SW_T8, SW_T9, SW_TASTA1, SW_TCOMMA1, SW_TDOT1, SW_TMINUS1, SW_TPLUS1, SW_TSLASH1, SW_U1, SW_UBAR1, SW_UP1, SW_V1, SW_W1, SW_X1, SW_Y1, SW_YEN1, SW_Z1: footprint 1-Keyboard:CherryMX_1.25U -> 1-Keyboard:CherryMX_1U
- SW_CLS1, SW_DEL1, SW_F1, SW_F2, SW_F3, SW_F4, SW_F5, SW_INS1, SW_SEL1, SW_STOP1, SW_TAB1: footprint 1-Keyboard:CherryMX_1.25U -> 1-Keyboard:CherryMX_1.5U
- SW_CTRL1: footprint 1-Keyboard:CherryMX_1.25U -> 1-Keyboard:CherryMX_2U
- SW_RET1: footprint 1-Keyboard:CherryMX_1.25U -> 1-Keyboard:CherryMX_ISO_Enter
- SW_SFT1, SW_SFT2: footprint 1-Keyboard:CherryMX_1.25U -> 1-Keyboard:CherryMX_2.5U
- SW_SPC1: footprint 1-Keyboard:CherryMX_1.25U -> 1-Keyboard:CherryMX_6U
- moved SW_SFT1 13.5 mm to (81.0, 200.5)
- moved SW_F1 12.6 mm to (71.4, 112.3)
- moved SW_CTRL1 8.91 mm to (76.4, 178.1)
- moved SW_F2 8.75 mm to (100.6, 112.3)
- moved SW_F3 5.19 mm to (129.6, 112.3)
- moved SW_SFT2 4.81 mm to (402.4, 200.5)
- moved SW_UBAR1 4.81 mm to (366.8, 200.5)
- moved SW_CLS1 4.33 mm to (280.7, 112.3)
- moved SW_TAB1 4.21 mm to (71.7, 155.8)
- moved SW_SEL1 4.18 mm to (350.3, 111.5)
- moved SW_DEL1 3.57 mm to (408.2, 111.5)
- moved SW_RET1 3.27 mm to (414.1, 165.5)
- moved SW_F4 1.77 mm to (158.4, 112.3)
- moved SW_F5 1.67 mm to (187.3, 112.3)
- moved SW_SLASH1 1.64 mm to (344.6, 200.5)
Routing:
- net /X5: track 810.7 -> 822.8 mm
- net /X7: track 790.5 -> 800.8 mm
- net /X6: track 745.8 -> 755.5 mm
- net Net-(D9-A): track 558.8 -> 565.9 mm
- net /X0: track 881.4 -> 874.8 mm
- net Net-(D7-A): track 657.8 -> 652.8 mm
- net /X4: track 829.6 -> 834.1 mm
- net VCC: track 444.0 -> 448.5 mm
- net Net-(D8-A): track 446.7 -> 449.4 mm
- net Net-(D3-A): track 451.1 -> 448.4 mm
- net /X3: track 770.2 -> 768.3 mm
- net /X2: track 761.2 -> 759.5 mm
