File: projects/msx_keyboard/msx_keyboard.kicad_sch (KiCad schematic)
At the start: 111 parts, among them J1 Conn_01x04_Pin, J2 Conn_01x08_Pin, U1 4515

Commit message: Updated
Parts:
- added D12: CAPS_LED, LED_THT:LED_D5.0mm, symbol Device:LED
- added D13: KANA_LED, LED_THT:LED_D5.0mm, symbol Device:LED
- added J3, J4: Conn_01x01_Pin, Connector_PinSocket_2.54mm:PinSocket_1x01_P2.54mm_Vertical, symbol Connector:Conn_01x01_Pin
- added J5: Conn_01x02_Pin, Connector_PinHeader_2.54mm:PinHeader_1x02_P2.54mm_Vertical, symbol Connector:Conn_01x02_Pin
- added R10, R9: R, Resistor_THT:R_Axial_DIN0207_L6.3mm_D2.5mm_P7.62mm_Horizontal, symbol Device:R
Connections:
- net GND: now also J5.2 (Pin_2)
- net VCC: now also J5.1 (Pin_1), R10.1, R9.1
- new net: D13.1 (K), J4.1 (Pin_1)
- new net: D12.1 (K), J3.1 (Pin_1)
- new net: D12.2 (A), R10.2
- new net: D13.2 (A), R9.2
Other:
- note added: "PPI PC6"
- note added: "PSG IOB7"

Commit message: Updated
Parts:
- added C1: C, Capacitor_THT:C_Disc_D3.0mm_W1.6mm_P2.50mm, symbol Device:C
- SW_0, SW_1, SW_2, SW_3, SW_4, SW_5, SW_6, SW_7, SW_8, SW_9, SW_A1, SW_ASTA1, SW_AT1, SW_B1, SW_BS1, SW_C1, SW_CAPS1, SW_D1, SW_DOWN1, SW_E1, SW_ESC1, SW_F6, SW_G1, SW_GRP1, SW_GT1, SW_H1, SW_HAT1, SW_I1, SW_J1, SW_K1, SW_KANA1, SW_L1, SW_LBRAC1, SW_LEFT1, SW_LT1, SW_M1, SW_MINUS1, SW_N1, SW_O1, SW_P1, SW_PLUS1, SW_Q1, SW_R1, SW_RBRAC1, SW_RIGHT1, SW_S1, SW_SLASH1, SW_T0, SW_T1, SW_T10, SW_T2, SW_T3, SW_T4, SW_T5, SW_T6, SW_T7, SW_T8, SW_T9, SW_TASTA1, SW_TCOMMA1, SW_TDOT1, SW_TMINUS1, SW_TPLUS1, SW_TSLASH1, SW_U1, SW_UBAR1, SW_UP1, SW_V1, SW_W1, SW_X1, SW_Y1, SW_YEN1, SW_Z1: footprint 1-Keyboard:CherryMX_1.25U -> 1-Keyboard:CherryMX_1U
- SW_CLS1, SW_DEL1, SW_F1, SW_F2, SW_F3, SW_F4, SW_F5, SW_INS1, SW_SEL1, SW_STOP1, SW_TAB1: footprint 1-Keyboard:CherryMX_1.25U -> 1-Keyboard:CherryMX_1.5U
- SW_CTRL1: footprint 1-Keyboard:CherryMX_1.25U -> 1-Keyboard:CherryMX_2U
- SW_RET1: footprint 1-Keyboard:CherryMX_1.25U -> 1-Keyboard:CherryMX_ISO_Enter
- SW_SFT1, SW_SFT2: footprint 1-Keyboard:CherryMX_1.25U -> 1-Keyboard:CherryMX_2.5U
- SW_SPC1: footprint 1-Keyboard:CherryMX_1.25U -> 1-Keyboard:CherryMX_6U
Connections:
- net GND: now also C1.2
- net VCC: now also C1.1
Other:
- note added: "パスコン"
